File: XT-IDE.kicad_sch (KiCad schematic)
At the start: 44 parts, among them J1 CONN_3, J2 CONN_3, J3 CONN_2, J4 CONN_2, J5 INTERRUPT, P6 CONN_1, P7 CONN_1, SW1 I/O ADDR, SW2 ROM OPT, U1 74LS573, U10 74LS688, U11 74LS245, U2 74LS573, U3 74LS245, U4 74LS04, U5 74LS32, U6 74LS04, U7 74LS138, U8 74LS688, U9 28C256

Commit message: WIP schematic cleanup, net renames, moving to global labels instead of wire labels, fixing polarities
Connections:
- net /ROM_WE is gone; now on net *WE_ROM: U9.27 (*WE)
- net *HI_BYTE_OUTPUT renamed *HI_WR_ENA
- net *HI_OUT_DELAYED renamed *HI_WR_DELAYED
- net *IOR-ISA renamed *BIOR
- net *IOW-ISA renamed *BIOW
- net *MEMR renamed *BMEMR
- net *MEMW renamed *BMEMW
- net /ROM_WE renamed *WE_ROM
- net 3 renamed HI_WR_LOAD
- net 4 renamed *HI_RD_ENA
- net 5 renamed HI_RD_LOAD
- net A0-ISA renamed BA0
- net A1-ISA renamed BA1
- net A10 renamed BA10
- net A11 renamed BA11
- net A12 renamed BA12
- net A13 renamed BA13
- net A14 renamed BA14
- net A15 renamed BA15
- net A16 renamed BA16
- net A17 renamed BA17
- net A18 renamed BA18
- net A19 renamed BA19
- net A2-ISA renamed BA2
- net A3 renamed BA3
- net A4 renamed BA4
- net A5 renamed BA5
- net A6 renamed BA6
- net A7 renamed BA7
- net A8 renamed BA8
- net A9 renamed BA9
- net AEN renamed BAEN
- net IRQ2 renamed BIRQ2
- net IRQ3 renamed BIRQ3
- net IRQ4 renamed BIRQ4
- net IRQ5 renamed BIRQ5
- net IRQ7 renamed BIRQ7
- net PC-DB0 renamed BD0
- net PC-DB1 renamed BD1
- net PC-DB2 renamed BD2
- net PC-DB3 renamed BD3
- net PC-DB4 renamed BD4
- net PC-DB5 renamed BD5
- net PC-DB6 renamed BD6
- net PC-DB7 renamed BD7
- net RESDRV renamed BRESET
- no-connect marks 23 -> 33
Other:
- moved on the sheet: P6, P7, U1, U2
