File: XT-IDE.kicad_pcb (KiCad board)
At the start: 2 copper layers, 114.3 x 106.7 mm, 46 parts, among them J1 CONN_3, J2 CONN_3, J3 CONN_2, J4 CONN_2, J5 INTERRUPT, P6 CONN_1, P7 CONN_1, SW1 I/O ADDR, SW2 ROM OPT, U1 74LS573, U10 74LS688, U11 74LS245, U2 74LS573, U3 74LS245, U4 74LS04, U5 74LS32, U6 74LS04, U7 74LS138, U8 74LS688, U9 28C256

Commit message: Add files via upload
Other:
- net class Default removed
- net class Power removed
- rule pad_to_mask_clearance: 0.254 -> 0
- board text added: "XT-IDE rev 05 (c) 2025 The Wizard http://www.TheWizard.cl/"
- board text added: "XT2IDE-5"
- board text added: "www.TheWizard.cl/"
- board text removed: "GW-XTIDE-4"
- board text removed: "XT-IDE rev 04 (c) 2017 The Glitch Works http://www.glitchwrks.com/xt-ide"
- board text removed: "www.glitchwrks.com/xt-ide"
